File: ScoreBoradPCB/ScoreBoradPCB.kicad_pcb (KiCad board)
At the start: 2 copper layers, 100 x 100 mm, 128 parts, among them J1 Conn_01x08_Male, J10 Conn_01x02_Male, J2 Conn_01x08_Male, J3 Conn_01x08_Male, J4 Conn_01x04_Male, J5 Conn_01x04_Male, J6 Conn_01x02_Male, J7 Conn_01x02_Male, J8 Conn_01x06_Male, J9 Conn_01x02_Male, Q1 2N7002K, Q10 NP52N06SLG, Q11 2N7002K, Q12 NP52N06SLG, Q13 2N7002K, Q14 NP52N06SLG, Q15 BSS84, Q16 NP52N06SLG, Q17 2N7002K, Q18 BSS84, Q19 NP52N06SLG, Q2 NP52N06SLG, Q20 2N7002K, Q21 BSS84, Q22 NP52N06SLG, Q23 2N7002K, Q24 2N7002K, Q3 2N7002K, Q4 NP52N06SLG, Q5 2N7002K, Q6 NP52N06SLG, Q7 2N7002K, Q8 NP52N06SLG, Q9 2N7002K, SW1 SW_Push, SW2 SW_Push, SW3 SW_Push, SW4 SW_Push, SW5 SW_Push, SW6 SW_Push, SW7 SW_Push, U1 PIC16F18854-SO, U2 TLP291, U3 IR2104, U4 TLP291, U5 IR2104, U6 TLP291, U7 IR2104

Commit message: 基板完成
Parts:
- added R44: 1k, Resistor_SMD:R_0603_1608Metric, F.Cu at (125.7, 88.3)
- added R45: 1k, Resistor_SMD:R_0603_1608Metric, F.Cu at (125.7, 92.1)
- R43: value 3k -> 1k
- U1: value PIC16F18854-SO -> PIC16F1938
- moved D10 2.54 mm to (137.8, 96.5)
- moved D11 2.54 mm to (141.6, 96.5)
- moved D7 2.54 mm to (125.7, 96.5)
- moved D8 2.54 mm to (129.5, 96.5)
- moved D9 2.54 mm to (133.3, 96.5)
- moved J7 2.01 mm to (194.9, 74.3)
- moved J5 2.01 mm to (194.9, 55.2)
- moved J6 1.91 mm to (106.7, 74.3)
- moved R60 1.91 mm to (103.5, 74.3)
- moved J4 1.90 mm to (106.7, 55.2)
- moved R61 1.90 mm to (103.5, 76.8)
- moved Q1 1.27 mm to (113.0, 142.9)
- moved Q11 1.27 mm to (182.9, 142.9)
- moved Q13 1.27 mm to (196.8, 142.9)
- moved Q3 1.27 mm to (127.0, 142.9)
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- renumbered R44 to R46, R45 to R47, R46 to R48, R47 to R49, R48 to R50, R49 to R62, R50 to R63
Connections:
- J2 pad 1: /Anode_one -> /Anode_ten
- J3 pad 1: /Anode_one -> /Anode_hun
- R43 pad 2: Net-(D7-Pad2) -> Net-(R43-Pad2)
- R63 pad 1: +12V -> Net-(Q24-Pad3)
- R63 pad 2: Net-(Q24-Pad3) -> +12V
Routing:
- net GND: track 0.00 -> 581.6 mm, vias 0 -> 18
- net +12V: track 0.00 -> 360.8 mm, vias 0 -> 2
- net +5V: track 0.00 -> 237.7 mm, vias 0 -> 1
- net +48V: track 0.00 -> 231.9 mm
- net /SCL: track 0.00 -> 164.3 mm, vias 0 -> 1
- net /SDA: track 0.00 -> 159.0 mm, vias 0 -> 1
- net /Cathode_a: track 0.00 -> 122.0 mm
- net /Cathode_b: track 0.00 -> 113.8 mm
- net /Cathode_c: track 0.00 -> 102.8 mm
- net /Segment_g: track 0.00 -> 100.4 mm, vias 0 -> 1
- net /Cathode_d: track 0.00 -> 93.3 mm
- net /Plus_one: track 0.00 -> 92.4 mm, vias 0 -> 1
- net Net-(Q24-Pad3): track 0.00 -> 90.0 mm
- net /Segment_f: track 0.00 -> 89.5 mm, vias 0 -> 1
- net /Cathode_e: track 0.00 -> 83.9 mm
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- added copper zone on B.Cu, net GND
- added copper zone on F.Cu, net GND
Other:
- board text added: "+1"
- board text added: "+10"
- board text added: "+100"
- board text added: "+12V"
- board text added: "+48V"
- board text added: "+48v +5V +12V GND"
- board text added: "+5V"
- board text added: "-1"
- board text added: "-10"
- board text added: "-100"
- board text added: "1"
- board text added: "10"
- board text added: "100"
- board text added: "LED"
- board text added: "LED_OFF"
- board text added: "SDA SCL"
- board text added: "com a b c d e f g"

Commit message: 校訓追加
Parts:
- added G***: LOGO, logo:Koukun, F.Cu at (151.1, 108.0)

Commit message: パターン完成
Parts:
- removed D11: LED, LED_SMD:LED_0603_1608Metric
- removed R50: 300, Resistor_SMD:R_0603_1608Metric
- moved D9 46.3 mm to (175.3, 76.8)
- moved D10 45.7 mm to (179.1, 76.8)
- moved D8 45.7 mm to (170.8, 76.8)
- moved R47 44.2 mm to (170.8, 72.4)
- moved R48 43.6 mm to (175.3, 72.4)
- moved D7 43.4 mm to (164.5, 76.8)
- moved R45 43.4 mm to (164.5, 72.4)
- moved R49 43.0 mm to (179.1, 72.4)
- moved R46 41.2 mm to (168.9, 72.4)
- moved R44 40.1 mm to (162.6, 72.4)
- moved R43 37.0 mm to (160.7, 72.4)
- moved G*** 13.7 mm to (138.4, 113.0)
- moved Q5 0.64 mm to (141.0, 143.5)
- moved Q9 0.64 mm to (168.9, 143.5)
- moved Q1 0.63 mm to (113.0, 142.2)
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Connections:
- U1 pad 18: /LED -> Net-(U1-Pad18)
Routing:
- net /ShutDown: track 60.7 -> 127.4 mm
- net /LED: track 62.1 -> 0.00 mm, vias 1 -> 0
- net +12V: track 360.8 -> 420.7 mm, vias 2 -> 1
- net +48V: track 231.9 -> 197.0 mm, vias 0 -> 1
- net /Plus_one: track 92.4 -> 66.7 mm, vias 1 -> 2
- net GND: track 581.6 -> 607.1 mm, vias 18 -> 7
- net /SCL: track 164.3 -> 143.8 mm, vias 1 -> 0
- net Net-(Q24-Pad3): track 90.0 -> 106.3 mm
- net /Segment_b: track 58.1 -> 70.7 mm
- net Net-(D11-Pad2): track 10.5 -> 0.00 mm
- net /Anode_ten: track 51.6 -> 43.3 mm
- net Net-(D10-Pad2): track 11.1 -> 2.87 mm
- net Net-(D9-Pad2): track 10.5 -> 2.87 mm
- net +5V: track 237.7 -> 243.9 mm
- net /Minus_hun: track 32.8 -> 38.7 mm
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Other:
- board text added: "RST"
- board text added: "SD"
- board text removed: "LED"
- board text removed: "LED_OFF"
