File: ScoreBoradPCB/ScoreBoradPCB.sch (KiCad schematic (older format))
At the start: 1 part, among them U1 PIC16F18854-SO

Commit message: フットプリント配置完了
Parts:
- added C1, C2, C4, C6: 0.1u, Capacitor_SMD:C_0603_1608Metric, symbol Device:C
- added C3, C5, C7: 10u, Capacitor_SMD:C_0603_1608Metric, symbol Device:C_Small
- added D1, D2, D3, D4, D5, D6: GS1010FL, Diode_SMD:D_SOD-123F, symbol Device:D
- added D10, D11, D7, D8, D9: LED, LED_SMD:LED_0603_1608Metric, symbol Device:LED
- added DS1: 2831BS-RIGHT-ANGLE, 2831BS-RIGHT-ANGLE:DIPS762W45P254L2253H610Q12N, symbol 2831BS-RIGHT-ANGLE:2831BS-RIGHT-ANGLE
- added J1, J2, J3: Conn_01x08_Male, Connector_JST:JST_VH_B8P-VH_1x08_P3.96mm_Vertical, symbol Connector:Conn_01x08_Male
- added J10, J9: Conn_01x02_Male, Connector_PinHeader_2.54mm:PinHeader_1x02_P2.54mm_Vertical, symbol Connector:Conn_01x02_Male
- added J4, J5: Conn_01x04_Male, Connector_JST:JST_VH_B4P-VH_1x04_P3.96mm_Vertical, symbol Connector:Conn_01x04_Male
- added J6, J7: Conn_01x02_Male, Connector_JST:JST_XH_B2B-XH-A_1x02_P2.50mm_Vertical, symbol Connector:Conn_01x02_Male
- added J8: Conn_01x06_Male, Connector_PinHeader_2.54mm:PinHeader_1x06_P2.54mm_Horizontal, symbol Connector:Conn_01x06_Male
- added Q1, Q11, Q13, Q17, Q20, Q23, Q24, Q3, Q5, Q7, Q9: 2N7002K, Package_TO_SOT_SMD:SOT-23, symbol Device:Q_NMOS_GSD
- added Q10, Q12, Q14, Q16, Q19, Q2, Q22, Q4, Q6, Q8: NP52N06SLG, Package_TO_SOT_SMD:TO-252-3_TabPin4, symbol Device:Q_NMOS_GDSD
- added Q15, Q18, Q21: BSS84, Package_TO_SOT_SMD:SOT-23, symbol Device:Q_PMOS_GSD
- added R1, R10, R13, R16, R19, R25, R26, R32, R33, R39, R4, R40, R7: 100, Resistor_SMD:R_0603_1608Metric, symbol Device:R
- added R11, R12, R14, R15, R17, R18, R2, R20, R21, R22, R24, R27, R28, R29, R3, R31, R34, R35, R36, R38, R41, R42, R49, R5, R50, R58, R59, R6, R8, R9: 15k, Resistor_SMD:R_0603_1608Metric, symbol Device:R
- added R23, R30, R37, R44, R45, R46, R47, R48, R51, R52, R53, R54, R55, R56, R57: 300, Resistor_SMD:R_0603_1608Metric, symbol Device:R
- added R43: 3k, Resistor_SMD:R_0603_1608Metric, symbol Device:R
- added R60, R61: 1k, Resistor_SMD:R_0603_1608Metric, symbol Device:R
- added SW1, SW2, SW3, SW4, SW5, SW6, SW7: SW_Push, Button_Switch_THT:SW_PUSH_6mm_H5mm, symbol Switch:SW_Push
- added U2, U4, U6: TLP291, Package_SO:SOIC-4_4.55x2.6mm_P1.27mm, symbol Isolator:TLP291
- added U3, U5, U7: IR2104, Package_SO:SOIC-8_3.9x4.9mm_P1.27mm, symbol Driver_FET:IR2104
- U1: footprint Package_SO:SOIC-28W_7.5x17.9mm_P1.27mm -> Package_DIP:DIP-28_W7.62mm_Socket
Connections:
- net GND: now also C1.2, C2.2, C4.2, C6.2, D10.1 (K), D11.1 (K), D7.1 (K), D8.1 (K), D9.1 (K), J4.4 (Pin_4), J5.4 (Pin_4), J8.4 (Pin_4), Q1.2 (S), Q10.3 (S), Q11.2 (S), Q12.3 (S), Q13.2 (S), Q14.3 (S), Q17.2 (S), Q2.3 (S), Q20.2 (S), Q23.2 (S), Q24.2 (S), Q3.2 (S), Q4.3 (S), Q5.2 (S), Q6.3 (S), Q7.2 (S), Q8.3 (S), Q9.2 (S), R11.1, R14.1, R17.1, R2.1, R20.1, R24.2, R28.1, R31.2, R35.1, R38.2, R42.1, R49.2, R5.1, R58.2, R59.2, R8.1, SW1.1, SW2.1, SW3.1, SW4.1, SW5.1, SW6.1, SW7.1, U2.2, U3.4 (COM), U4.2, U5.4 (COM), U6.2, U7.4 (COM)
- net Vpp_MCLR: now reaches U1.1 (VPP/~MCLR/RE3)
- net Vpp_MCLR: now also J8.6 (Pin_6), SW7.2
- net Segment_g: now reaches U1.10 (RA6)
- net Segment_g: now also R19.2
- net Place_one: now reaches U1.11 (RC0)
- net Place_one: now also Q15.1 (G), R22.2
- net Place_ten: now reaches U1.12 (RC1)
- net Place_ten: now also Q18.1 (G), R29.2
- net Place_hun: now reaches U1.13 (RC2)
- net Place_hun: now also Q21.1 (G), R36.2
- net SCL: now reaches U1.14 (RC3)
- net SCL: now also J6.2 (Pin_2), J7.2 (Pin_2), R61.2
- net SDA: now reaches U1.15 (RC4)
- net SDA: now also J6.1 (Pin_1), J7.1 (Pin_1), R60.2
- net Address_1: now reaches U1.16 (RC5)
- net Address_1: now also J9.2 (Pin_2), R58.1
- net Address_2: now reaches U1.17 (RC6)
- net Address_2: now also J10.2 (Pin_2), R59.1
- net LED: now reaches U1.18 (RC7)
- net LED: now also R48.1
- net Segment_a: now reaches U1.2 (RA0)
- net Segment_a: now also R1.2
- net +5V: now reaches U1.20 (VDD)
- net +5V: now also C1.1, J10.1 (Pin_1), J4.2 (Pin_2), J5.2 (Pin_2), J8.5 (Pin_5), J9.1 (Pin_1), Q15.2 (S), Q18.2 (S), Q21.2 (S), R22.1, R29.1, R36.1, R46.1, R60.1, R61.1
- net Plus_one: now reaches U1.21 (RB0)
- net Plus_one: now also SW6.2
- net Minus_one: now reaches U1.22 (RB1)
- net Minus_one: now also SW5.2
- net Plus_ten: now reaches U1.23 (RB2)
- net Plus_ten: now also SW4.2
- net Minus_ten: now reaches U1.24 (RB3)
- net Minus_ten: now also SW3.2
- net Plus_hun: now reaches U1.25 (RB4)
- net Plus_hun: now also SW2.2
- net Minus_hun: now reaches U1.26 (RB5)
- net Minus_hun: now also SW1.2
- net ICSP_CLK: now reaches U1.27 (RB6)
- net ICSP_CLK: now also J8.2 (Pin_2)
- net ICSP_DAT: now reaches U1.28 (RB7)
- net ICSP_DAT: now also J8.3 (Pin_3)
- net Segment_b: now reaches U1.3 (RA1)
- net Segment_b: now also R4.2
- net Segment_c: now reaches U1.4 (RA2)
- net Segment_c: now also R7.2
- net Segment_d: now reaches U1.5 (RA3)
- net Segment_d: now also R10.2
- net Segment_e: now reaches U1.6 (RA4)
- net Segment_e: now also R13.2
- net Segment_f: now reaches U1.7 (RA5)
- net Segment_f: now also R16.2
- net ShutDown: now reaches U1.9 (RA7)
- net ShutDown: now also Q24.1 (G), R47.1, R49.1
- new net: Q1.3 (D), Q2.1 (G), R3.2
- new net: Q1.1 (G), R1.1, R2.2
- new net: Q3.1 (G), R4.1, R5.2
- new net: Q3.3 (D), Q4.1 (G), R6.2
- new net: Q5.1 (G), R7.1, R8.2
- new net: Q5.3 (D), Q6.1 (G), R9.2
- new net: Q7.1 (G), R10.1, R11.2
- new net: Q7.3 (D), Q8.1 (G), R12.2
- new net: Q9.1 (G), R13.1, R14.2
- new net: Q10.1 (G), Q9.3 (D), R15.2
- new net: Q11.1 (G), R16.1, R17.2
- new net: Q11.3 (D), Q12.1 (G), R18.2
- new net: Q13.1 (G), R19.1, R20.2
- new net: Q13.3 (D), Q14.1 (G), R21.2
- new net: D1.2 (A), Q15.3 (D), R23.2
- new net: R23.1, U2.1
- new net: R24.1, U2.3, U3.2 (IN)
- new net: Q24.3 (D), R50.2, U3.3 (~SD), U5.3 (~SD), U7.3 (~SD)
- new net: R26.2, U3.5 (LO)
- new net: R25.2, U3.7 (HO)
- new net: C3.1, D2.1 (K), U3.8 (VB)
- new net: Q16.1 (G), R25.1, R27.2
- new net: Q17.1 (G), R26.1, R28.2
- new net: D3.2 (A), Q18.3 (D), R30.2
- new net: R30.1, U4.1
- new net: R31.1, U4.3, U5.2 (IN)
- new net: R33.2, U5.5 (LO)
- new net: R32.2, U5.7 (HO)
- new net: C5.1, D4.1 (K), U5.8 (VB)
- new net: Q20.1 (G), R33.1, R35.2
- new net: Q19.1 (G), R32.1, R34.2
- new net: D5.2 (A), Q21.3 (D), R37.2
- new net: R37.1, U6.1
- new net: R38.1, U6.3, U7.2 (IN)
- new net: R40.2, U7.5 (LO)
- new net: R39.2, U7.7 (HO)
- new net: C7.1, D6.1 (K), U7.8 (VB)
- new net: Q23.1 (G), R40.1, R42.2
- new net: Q22.1 (G), R39.1, R41.2
- new net: D7.2 (A), R43.2
- new net: R44.2, R45.1
- new net: D8.2 (A), R45.2
- new net: D9.2 (A), R46.2
- new net: D10.2 (A), R47.2
- new net: D11.2 (A), R48.2
- new net: DS1.1 (CATHODE_E), R51.1
- new net: DS1.10 (CATHODE_F), R56.1
- new net: DS1.11 (CATHODE_A), R57.1
- new net: DS1.2 (CATHODE_D), R52.1
- new net: DS1.4 (CATHODE_C), R53.1
- new net: DS1.5 (CATHODE_G), R54.1
- new net: DS1.7 (CATHODE_B), R55.1
- new net +12V: C2.1, C4.1, C6.1, D2.2 (A), D4.2 (A), D6.2 (A), J4.3 (Pin_3), J5.3 (Pin_3), R12.1, R15.1, R18.1, R21.1, R3.1, R44.1, R50.1, R6.1, R9.1, U2.4, U3.1 (VCC), U4.4, U5.1 (VCC), U6.4, U7.1 (VCC)
- new net +48V: J4.1 (Pin_1), J5.1 (Pin_1), Q16.4 (D), Q19.4 (D), Q22.4 (D), R43.1
- new net Anode_hun: C7.2, Q22.3 (S), Q23.3 (D), R41.1, U7.6 (VS)
- new net Anode_one: C3.2, J1.1 (Pin_1), J2.1 (Pin_1), J3.1 (Pin_1), Q16.3 (S), Q17.3 (D), R27.1, U3.6 (VS)
- new net Anode_ten: C5.2, Q19.3 (S), Q20.3 (D), R34.1, U5.6 (VS)
- new net Cathode_a: J1.2 (Pin_2), J2.2 (Pin_2), J3.2 (Pin_2), Q2.4 (D), R57.2
- new net Cathode_b: J1.3 (Pin_3), J2.3 (Pin_3), J3.3 (Pin_3), Q4.4 (D), R55.2
- new net Cathode_c: J1.4 (Pin_4), J2.4 (Pin_4), J3.4 (Pin_4), Q6.4 (D), R53.2
- new net Cathode_d: J1.5 (Pin_5), J2.5 (Pin_5), J3.5 (Pin_5), Q8.4 (D), R52.2
- new net Cathode_e: J1.6 (Pin_6), J2.6 (Pin_6), J3.6 (Pin_6), Q10.4 (D), R51.2
- new net Cathode_f: J1.7 (Pin_7), J2.7 (Pin_7), J3.7 (Pin_7), Q12.4 (D), R56.2
- new net Cathode_g: J1.8 (Pin_8), J2.8 (Pin_8), J3.8 (Pin_8), Q14.4 (D), R54.2
- new net Dig_hun: D5.1 (K), DS1.12 (COMMON_ANODE_DIG_1)
- new net Dig_one: D1.1 (K), DS1.8 (COMMON_ANODE_DIG_3)
- new net Dig_ten: D3.1 (K), DS1.9 (COMMON_ANODE_DIG_2)
- no-connect marks 0 -> 12
Other:
- moved on the sheet: U1

Commit message: 基板完成
Parts:
- added R44, R45: 1k, Resistor_SMD:R_0603_1608Metric, symbol Device:R
- R43: value 3k -> 1k
- U1: value PIC16F18854-SO -> PIC16F1938
- renumbered R44 to R46, R45 to R47, R46 to R48, R47 to R49, R48 to R50, R49 to R62, R50 to R63
Connections:
- net +12V: now also R63.2; no longer R63.1
- net Anode_hun: now also J3.1 (Pin_1)
- net Anode_one: no longer J2.1 (Pin_1), J3.1 (Pin_1)
- net Anode_ten: now also J2.1 (Pin_1)
- net at Q24.3 (D), U3.3 (~SD), U5.3 (~SD)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: now also R63.1; no longer R63.2
- net at D7.2 (A): now also R45.2; no longer R43.2
- new net: R43.2, R44.1
- new net: R44.2, R45.1
Other:
- moved on the sheet: D10, D11, D7, D8, D9
Changed lines of the file:
@@
 P 2200 3900
 F 0 "U1" H 2200 4881 50  0000 C CNN
-F 1 "PIC16F18854-SO" H 2200 4790 50  0000 C CNN
+F 1 "PIC16F1938" H 2200 4790 50  0000 C CNN
 F 2 "Package_DIP:DIP-28_W7.62mm_Socket" H 2200 2800 50  0001 C CNN
-F 3 "http://ww1.microchip.com/downloads/en/DeviceDoc/PIC16(L)F18854%20Data%20Sheet_DS40001826C.pdf" H 2500 3300 50  0001 C CNN
+F 3 "https://akizukidenshi.com/download/pic16f193X.pdf" H 2500 3300 50  0001 C CNN
 	1    2200 3900
 	1    0    0    -1
@@
 ShutDown
 $Comp
-L Device:R R49
+L Device:R R62
 U 1 1 5F8A6840
 P 7250 10400
-F 0 "R49" H 7320 10446 50  0000 L CNN
+F 0 "R62" H 7320 10446 50  0000 L CNN
 F 1 "15k" H 7320 10355 50  0000 L CNN
 F 2 "Resistor_SMD:R_0603_1608Metric" V 7180 10400 50  0001 C CNN
@@
 	7600 10550 7600 10400
 $Comp
-L Device:R R50
+L Device:R R63
 U 1 1 5F8E0D1A
 P 7800 9950
-F 0 "R50" V 7593 9950 50  0000 C CNN
-F 1 "15k" V 7684 9950 50  0000 C CNN
+F 0 "R63" V 8007 9950 50  0000 C CNN
+F 1 "15k" V 7916 9950 50  0000 C CNN
 F 2 "Resistor_SMD:R_0603_1608Metric" V 7730 9950 50  0001 C CNN
 F 3 "~" H 7800 9950 50  0001 C CNN
 	1    7800 9950
-	0    1    1    0
+	0    -1   -1   0
 $EndComp
 Wire Wire Line
@@
 	7600 8900 7600 6650
 $Comp
-L Device:R R43
-U 1 1 5F95C342
-P 1050 8500
-F 0 "R43" H 1120 8546 50  0000 L CNN
-F 1 "3k" H 1120 8455 50  0000 L CNN
-F 2 "Resistor_SMD:R_0603_1608Metric" V 980 8500 50  0001 C CNN
-F 3 "~" H 1050 8500 50  0001 C CNN
-	1    1050 8500
-	1    0    0    -1
-$EndComp
-$Comp
-L Device:R R44
+L Device:R R46
 U 1 1 5F95D4E2
 P 1400 8500
-F 0 "R44" H 1470 8546 50  0000 L CNN
+F 0 "R46" H 1470 8546 50  0000 L CNN
 F 1 "300" H 1470 8455 50  0000 L CNN
 F 2 "Resistor_SMD:R_0603_1608Metric" V 1330 8500 50  0001 C CNN
@@
 $EndComp
 $Comp
-L Device:R R45
+L Device:R R47
 U 1 1 5F95D6BE
 P 1400 8850
-F 0 "R45" H 1470 8896 50  0000 L CNN
+F 0 "R47" H 1470 8896 50  0000 L CNN
 F 1 "300" H 1470 8805 50  0000 L CNN
 F 2 "Resistor_SMD:R_0603_1608Metric" V 1330 8850 50  0001 C CNN
@@
 $EndComp
 $Comp
-L Device:R R46
+L Device:R R48
 U 1 1 5F95DAD8
 P 1750 8500
-F 0 "R46" H 1820 8546 50  0000 L CNN
+F 0 "R48" H 1820 8546 50  0000 L CNN
 F 1 "300" H 1820 8455 50  0000 L CNN
 F 2 "Resistor_SMD:R_0603_1608Metric" V 1680 8500 50  0001 C CNN
@@
 $EndComp
 $Comp
-L Device:R R47
+L Device:R R49
 U 1 1 5F95E012
 P 2100 8500
-F 0 "R47" H 2170 8546 50  0000 L CNN
+F 0 "R49" H 2170 8546 50  0000 L CNN
 F 1 "300" H 2170 8455 50  0000 L CNN
 F 2 "Resistor_SMD:R_0603_1608Metric" V 2030 8500 50  0001 C CNN
@@
 $EndComp
 $Comp
-L Device:R R48
+L Device:R R50
 U 1 1 5F95E20C
 P 2450 8500
-F 0 "R48" H 2520 8546 50  0000 L CNN
+F 0 "R50" H 2520 8546 50  0000 L CNN
 F 1 "300" H 2520 8455 50  0000 L CNN
 F 2 "Resistor_SMD:R_0603_1608Metric" V 2380 8500 50  0001 C CNN
@@
 Wire Wire Line
 	2450 8150 2450 8350
-Wire Wire Line
-	2450 9200 2450 8650
-Wire Wire Line
-	2100 8650 2100 9200
-Wire Wire Line
-	1750 9200 1750 8650
-Wire Wire Line
-	1400 9000 1400 9200
-Wire Wire Line
-	1050 9200 1050 8650
 $Comp
 L power:GND #PWR061
 U 1 1 5FA5950D
-P 1050 9650
-F 0 "#PWR061" H 1050 9400 50  0001 C CNN
-F 1 "GND" H 1055 9477 50  0000 C CNN
-F 2 "" H 1050 9650 50  0001 C CNN
-F 3 "" H 1050 9650 50  0001 C CNN
-	1    1050 9650
+P 1050 10050
+F 0 "#PWR061" H 1050 9800 50  0001 C CNN
+F 1 "GND" H 1055 9877 50  0000 C CNN
+F 2 "" H 1050 10050 50  0001 C CNN
+F 3 "" H 1050 10050 50  0001 C CNN
+	1    1050 10050
 	1    0    0    -1
 $EndComp
@@
 L power:GND #PWR063
 U 1 1 5FA59893
-P 1400 9650
-F 0 "#PWR063" H 1400 9400 50  0001 C CNN
-F 1 "GND" H 1405 9477 50  0000 C CNN
-F 2 "" H 1400 9650 50  0001 C CNN
-F 3 "" H 1400 9650 50  0001 C CNN
-	1    1400 9650
+P 1400 10050
+F 0 "#PWR063" H 1400 9800 50  0001 C CNN
+F 1 "GND" H 1405 9877 50  0000 C CNN
+F 2 "" H 1400 10050 50  0001 C CNN
+F 3 "" H 1400 10050 50  0001 C CNN
+	1    1400 10050
 	1    0    0    -1
 $EndComp
@@
 L power:GND #PWR065
 U 1 1 5FA59AAE
-P 1750 9650
-F 0 "#PWR065" H 1750 9400 50  0001 C CNN
-F 1 "GND" H 1755 9477 50  0000 C CNN
-F 2 "" H 1750 9650 50  0001 C CNN
-F 3 "" H 1750 9650 50  0001 C CNN
-	1    1750 9650
+P 1750 10050
+F 0 "#PWR065" H 1750 9800 50  0001 C CNN
+F 1 "GND" H 1755 9877 50  0000 C CNN
+F 2 "" H 1750 10050 50  0001 C CNN
+F 3 "" H 1750 10050 50  0001 C CNN
+	1    1750 10050
 	1    0    0    -1
 $EndComp
@@
 L power:GND #PWR066
 U 1 1 5FA59C54
-P 2100 9650
-F 0 "#PWR066" H 2100 9400 50  0001 C CNN
-F 1 "GND" H 2105 9477 50  0000 C CNN
-F 2 "" H 2100 9650 50  0001 C CNN
-F 3 "" H 2100 9650 50  0001 C CNN
-	1    2100 9650
+P 2100 10050
+F 0 "#PWR066" H 2100 9800 50  0001 C CNN
+F 1 "GND" H 2105 9877 50  0000 C CNN
+F 2 "" H 2100 10050 50  0001 C CNN
+F 3 "" H 2100 10050 50  0001 C CNN
+	1    2100 10050
 	1    0    0    -1
 $EndComp
@@
 L power:GND #PWR067
 U 1 1 5FA59F0C
-P 2450 9650
-F 0 "#PWR067" H 2450 9400 50  0001 C CNN
-F 1 "GND" H 2455 9477 50  0000 C CNN
-F 2 "" H 2450 9650 50  0001 C CNN
-F 3 "" H 2450 9650 50  0001 C CNN
-	1    2450 9650
+P 2450 10050
+F 0 "#PWR067" H 2450 9800 50  0001 C CNN
+F 1 "GND" H 2455 9877 50  0000 C CNN
+F 2 "" H 2450 10050 50  0001 C CNN
+F 3 "" H 2450 10050 50  0001 C CNN
+	1    2450 10050
 	1    0    0    -1
 $EndComp
 Wire Wire Line
-	2450 9650 2450 9500
+	2450 10050 2450 9900
 Wire Wire Line
-	2100 9500 2100 9650
+	2100 9900 2100 10050
 Wire Wire Line
-	1750 9650 1750 9500
+	1750 10050 1750 9900
 Wire Wire Line
-	1400 9500 1400 9650
+	1400 9900 1400 10050
 Wire Wire Line
-	1050 9650 1050 9500
+	1050 10050 1050 9900
 $Comp
 L 2831BS-RIGHT-ANGLE:2831BS-RIGHT-ANGLE DS1
@@
 	15000 3600 14650 3600
 Text Label 15000 4700 1    50   ~ 0
-Anode_one
+Anode_ten
 Wire Wire Line
 	15000 4700 15000 4750
@@
 	15000 4750 14650 4750
 Text Label 15000 5900 1    50   ~ 0
-Anode_one
+Anode_hun
 Wire Wire Line
 	15000 5900 15000 5950
@@
 L Device:LED D7
 U 1 1 60D8C192
-P 1050 9350
-F 0 "D7" V 1089 9232 50  0000 R CNN
-F 1 "LED" V 998 9232 50  0000 R CNN
-F 2 "LED_SMD:LED_0603_1608Metric" H 1050 9350 50  0001 C CNN
-F 3 "~" H 1050 9350 50  0001 C CNN
-	1    1050 9350
+P 1050 9750
+F 0 "D7" V 1089 9632 50  0000 R CNN
+F 1 "LED" V 998 9632 50  0000 R CNN
+F 2 "LED_SMD:LED_0603_1608Metric" H 1050 9750 50  0001 C CNN
+F 3 "~" H 1050 9750 50  0001 C CNN
+	1    1050 9750
 	0    -1   -1   0
 $EndComp
@@
 L Device:LED D8
 U 1 1 60D8D760
-P 1400 9350
-F 0 "D8" V 1439 9232 50  0000 R CNN
-F 1 "LED" V 1348 9232 50  0000 R CNN
-F 2 "LED_SMD:LED_0603_1608Metric" H 1400 9350 50  0001 C CNN
-F 3 "~" H 1400 9350 50  0001 C CNN
-	1    1400 9350
+P 1400 9750
+F 0 "D8" V 1439 9632 50  0000 R CNN
+F 1 "LED" V 1348 9632 50  0000 R CNN
+F 2 "LED_SMD:LED_0603_1608Metric" H 1400 9750 50  0001 C CNN
+F 3 "~" H 1400 9750 50  0001 C CNN
+	1    1400 9750
 	0    -1   -1   0
 $EndComp
@@
 L Device:LED D9
 U 1 1 60D8DA0E
-P 1750 9350
-F 0 "D9" V 1789 9232 50  0000 R CNN
-F 1 "LED" V 1698 9232 50  0000 R CNN
-F 2 "LED_SMD:LED_0603_1608Metric" H 1750 9350 50  0001 C CNN
-F 3 "~" H 1750 9350 50  0001 C CNN
-	1    1750 9350
+P 1750 9750
+F 0 "D9" V 1789 9632 50  0000 R CNN
+F 1 "LED" V 1698 9632 50  0000 R CNN
+F 2 "LED_SMD:LED_0603_1608Metric" H 1750 9750 50  0001 C CNN
+F 3 "~" H 1750 9750 50  0001 C CNN
+	1    1750 9750
 	0    -1   -1   0
 $EndComp
@@
 L Device:LED D10
 U 1 1 60D8DD79
-P 2100 9350
-F 0 "D10" V 2139 9232 50  0000 R CNN
-F 1 "LED" V 2048 9232 50  0000 R CNN
-F 2 "LED_SMD:LED_0603_1608Metric" H 2100 9350 50  0001 C CNN
-F 3 "~" H 2100 9350 50  0001 C CNN
-	1    2100 9350
+P 2100 9750
+F 0 "D10" V 2139 9632 50  0000 R CNN
+F 1 "LED" V 2048 9632 50  0000 R CNN
+F 2 "LED_SMD:LED_0603_1608Metric" H 2100 9750 50  0001 C CNN
+F 3 "~" H 2100 9750 50  0001 C CNN
+	1    2100 9750
 	0    -1   -1   0
 $EndComp
@@
 L Device:LED D11
 U 1 1 60D8E0D0
-P 2450 9350
-F 0 "D11" V 2489 9232 50  0000 R CNN
-F 1 "LED" V 2398 9232 50  0000 R CNN
-F 2 "LED_SMD:LED_0603_1608Metric" H 2450 9350 50  0001 C CNN
-F 3 "~" H 2450 9350 50  0001 C CNN
-	1    2450 9350
+P 2450 9750
+F 0 "D11" V 2489 9632 50  0000 R CNN
+F 1 "LED" V 2398 9632 50  0000 R CNN
+F 2 "LED_SMD:LED_0603_1608Metric" H 2450 9750 50  0001 C CNN
+F 3 "~" H 2450 9750 50  0001 C CNN
+	1    2450 9750
 	0    -1   -1   0
 $EndComp
+$Comp
+L Device:R R43
+U 1 1 6124C8BD
+P 1050 8500
+F 0 "R43" H 1120 8546 50  0000 L CNN
+F 1 "1k" H 1120 8455 50  0000 L CNN
+F 2 "Resistor_SMD:R_0603_1608Metric" V 980 8500 50  0001 C CNN
+F 3 "~" H 1050 8500 50  0001 C CNN
+	1    1050 8500
+	1    0    0    -1
+$EndComp
+$Comp
+L Device:R R44
+U 1 1 6124DB08
+P 1050 8850
+F 0 "R44" H 1120 8896 50  0000 L CNN
+F 1 "1k" H 1120 8805 50  0000 L CNN
+F 2 "Resistor_SMD:R_0603_1608Metric" V 980 8850 50  0001 C CNN
+F 3 "~" H 1050 8850 50  0001 C CNN
+	1    1050 8850
+	1    0    0    -1
+$EndComp
+$Comp
+L Device:R R45
+U 1 1 6127BA71
+P 1050 9200
+F 0 "R45" H 1120 9246 50  0000 L CNN
+F 1 "1k" H 1120 9155 50  0000 L CNN
+F 2 "Resistor_SMD:R_0603_1608Metric" V 980 9200 50  0001 C CNN
+F 3 "~" H 1050 9200 50  0001 C CNN
+	1    1050 9200
+	1    0    0    -1
+$EndComp
+Wire Wire Line
+	1050 8650 1050 8700
+Wire Wire Line
+	1050 9000 1050 9050
+Wire Wire Line
+	1050 9350 1050 9600
+Wire Wire Line
+	1400 9000 1400 9600
+Wire Wire Line
+	1750 8650 1750 9600
+Wire Wire Line
+	2100 8650 2100 9600
+Wire Wire Line
+	2450 8650 2450 9600
 $EndSCHEMATC

Commit message: パターン完成
Parts:
- removed D11: LED, LED_SMD:LED_0603_1608Metric, symbol Device:LED
- removed R50: 300, Resistor_SMD:R_0603_1608Metric, symbol Device:R
Connections:
- net LED: no longer names the net of U1.18 (RC7)
- no-connect marks 12 -> 13
Changed lines of the file:
@@
 Text Label 2800 4300 0    50   ~ 0
 Address_2
-Text Label 2800 4200 0    50   ~ 0
-LED
-Wire Wire Line
-	2700 4200 2800 4200
 Wire Wire Line
 	2700 4300 2800 4300
@@
 $EndComp
 $Comp
-L Device:R R50
-U 1 1 5F95E20C
-P 2450 8500
-F 0 "R50" H 2520 8546 50  0000 L CNN
-F 1 "300" H 2520 8455 50  0000 L CNN
-F 2 "Resistor_SMD:R_0603_1608Metric" V 2380 8500 50  0001 C CNN
-F 3 "~" H 2450 8500 50  0001 C CNN
-	1    2450 8500
-	1    0    0    -1
-$EndComp
-$Comp
 L power:+48V #PWR060
 U 1 1 5F960D39
@@
 Wire Wire Line
 	2100 8150 2100 8350
-Text Label 2450 8150 1    50   ~ 0
-LED
-Wire Wire Line
-	2450 8150 2450 8350
 $Comp
 L power:GND #PWR061
@@
 	1    0    0    -1
 $EndComp
-$Comp
-L power:GND #PWR067
-U 1 1 5FA59F0C
-P 2450 10050
-F 0 "#PWR067" H 2450 9800 50  0001 C CNN
-F 1 "GND" H 2455 9877 50  0000 C CNN
-F 2 "" H 2450 10050 50  0001 C CNN
-F 3 "" H 2450 10050 50  0001 C CNN
-	1    2450 10050
-	1    0    0    -1
-$EndComp
-Wire Wire Line
-	2450 10050 2450 9900
 Wire Wire Line
 	2100 9900 2100 10050
@@
 $EndComp
 $Comp
-L Device:LED D11
-U 1 1 60D8E0D0
-P 2450 9750
-F 0 "D11" V 2489 9632 50  0000 R CNN
-F 1 "LED" V 2398 9632 50  0000 R CNN
-F 2 "LED_SMD:LED_0603_1608Metric" H 2450 9750 50  0001 C CNN
-F 3 "~" H 2450 9750 50  0001 C CNN
-	1    2450 9750
-	0    -1   -1   0
-$EndComp
-$Comp
 L Device:R R43
 U 1 1 6124C8BD
@@
 Wire Wire Line
 	2100 8650 2100 9600
-Wire Wire Line
-	2450 8650 2450 9600
+NoConn ~ 2700 4200
 $EndSCHEMATC
