File: ControllerPCB/ControllerPCB.sch (KiCad schematic (older format))
At the start: 18 parts

Commit message: twe-liteテストコード
Connections:
- net GND: now also J?.14 (Pin_14)
- net ShutDown: now also J?.8 (Pin_8); no longer J?.10 (Pin_10)
- net roll_start: now also J?.9 (Pin_9); no longer J?.11 (Pin_11)
- net stop_hun: now also J?.13 (Pin_13); no longer J?.14 (Pin_14)
- net stop_one: now also J?.11 (Pin_11); no longer J?.12 (Pin_12)
- net stop_ten: now also J?.12 (Pin_12); no longer J?.13 (Pin_13)
- no-connect marks 1 -> 8
Changed lines of the file:
@@
 	0    1    1    0
 $EndComp
-Text Label 2100 5800 2    50   ~ 0
+Text Label 2100 5700 2    50   ~ 0
 stop_hun
-Text Label 2100 5700 2    50   ~ 0
+Text Label 2100 5600 2    50   ~ 0
 stop_ten
-Text Label 2100 5600 2    50   ~ 0
+Text Label 2100 5500 2    50   ~ 0
 stop_one
-Text Label 2100 5500 2    50   ~ 0
+Text Label 2100 5300 2    50   ~ 0
 roll_start
-Text Label 2100 5400 2    50   ~ 0
+Text Label 2100 5200 2    50   ~ 0
 ShutDown
 Wire Wire Line
-	2200 5800 2100 5800
+	2200 5700 2100 5700
 Wire Wire Line
-	2100 5700 2200 5700
+	2100 5600 2200 5600
 Wire Wire Line
-	2200 5600 2100 5600
+	2200 5500 2100 5500
 Wire Wire Line
-	2100 5500 2200 5500
+	2100 5300 2200 5300
 Wire Wire Line
-	2200 5400 2100 5400
+	2200 5200 2100 5200
+Wire Wire Line
+	1700 5800 2200 5800
+Wire Wire Line
+	1700 5900 1700 5800
+$Comp
+L power:GND #PWR?
+U 1 1 5F550DF4
+P 1700 5900
+F 0 "#PWR?" H 1700 5650 50  0001 C CNN
+F 1 "GND" H 1705 5727 50  0000 C CNN
+F 2 "" H 1700 5900 50  0001 C CNN
+F 3 "" H 1700 5900 50  0001 C CNN
+	1    1700 5900
+	1    0    0    -1
+$EndComp
+NoConn ~ 2200 5400
+NoConn ~ 2200 5000
+NoConn ~ 2200 5100
+NoConn ~ 2200 4700
+NoConn ~ 2700 5200
+NoConn ~ 2700 5100
+NoConn ~ 2700 4900
 $EndSCHEMATC

Commit message: 通信基板回路完成
Parts:
- added D1, D2: LED, LED_SMD:LED_0603_1608Metric, symbol Device:LED
- added R5, R6: 300, Resistor_SMD:R_0603_1608Metric, symbol Device:R
- added SW1: SW_Push, Button_Switch_THT:SW_PUSH_6mm_H5mm, symbol Switch:SW_Push
- C1, C2: renamed from C?; footprint (none) -> Capacitor_THT:CP_Radial_D5.0mm_P2.00mm
- J1, J4: renamed from J?; footprint (none) -> Connector_JST:JST_VH_B4P-VH_1x04_P3.96mm_Vertical
- J2, J5: renamed from J?; footprint (none) -> Connector_JST:JST_XH_B2B-XH-A_1x02_P2.50mm_Vertical
- J3: renamed from J?; footprint (none) -> Package_DIP:DIP-28_W15.24mm
- J6: renamed from J?; value Conn_02x04_Counter_Clockwise -> AE-PCA9306; footprint (none) -> Package_DIP:DIP-8_W7.62mm
- R1, R2, R3, R4: renamed from R?; footprint (none) -> Resistor_SMD:R_0603_1608Metric
- SW2, SW3, SW4, SW5, SW6: renamed from SW?; footprint (none) -> Button_Switch_THT:SW_PUSH_6mm_H5mm
- U1: renamed from U?; value LM2931-3.3_TO220 -> LM2940T-3.3
Connections:
- net GND: now also D1.1 (K), D2.1 (K), SW1.1
- net ShutDown: now also J3.13 (Pin_13); no longer J3.8 (Pin_8)
- net roll_start: now also J3.15 (Pin_15); no longer J3.9 (Pin_9)
- net stop_hun: now also J3.18 (Pin_18); no longer J3.13 (Pin_13)
- net stop_one: now also J3.16 (Pin_16); no longer J3.11 (Pin_11)
- net stop_ten: now also J3.17 (Pin_17); no longer J3.12 (Pin_12)
- net RESET: now reaches J3.21 (Pin_21)
- net RESET: now also SW1.2
- new net: D1.2 (A), R5.2
- new net: D2.2 (A), R6.2
- new net LED_ShutDown: J3.11 (Pin_11), R6.1
- new net LED_roll: J3.12 (Pin_12), R5.1
- no-connect marks 8 -> 16
